File: Hardware/BMS.kicad_sch (KiCad schematic)
At the start: 1 part, among them U1 STM32F091RCTx

Commit message: Hardware Schematics Added
Parts:
- removed U1: STM32F091RCTx, Package_QFP:LQFP-64_10x10mm_P0.5mm, symbol MCU_ST_STM32F0:STM32F091RCTx
- added C1, C10, C11, C12, C13, C14, C15, C16, C17, C18, C19, C2, C20, C21, C22, C23, C24, C25, C26, C27, C28, C29, C3, C30, C31, C32, C33, C34, C4, C5, C6, C7, C8, C9: 0.47uF, symbol Device:C_Small
- added C35, C38, C39, C40: 1uF, symbol Device:C_Small
- added C36, C37: 0.1uF, symbol Device:C_Small
- added C41: 0.22uF, symbol Device:C
- added J15?: Conn_01x22, symbol Connector_Generic:Conn_01x22
- added J?: Conn_01x02, symbol Connector_Generic:Conn_01x02
- added J?: Daisy-chain communication pins, symbol Connector_Generic:Conn_01x04
- added Q?: NPN, symbol Simulation_SPICE:NPN
- added R1, R11, R13, R15, R17, R19, R21, R23, R25, R27, R29, R3, R31, R33, R5, R7, R9: 10, symbol Device:R_US
- added R10, R12, R14, R16, R18, R2, R20, R22, R24, R26, R28, R30, R32, R34, R4, R41, R6, R8: 100, symbol Device:R_US
- added R35, R36, R37, R38, R39, R40: 10.0k, symbol Device:R_US
- added R42: 200, symbol Device:R_US
- added RT1, RT2, RT3, RT4, RT5, RT6: T*, symbol Connector_Generic:Conn_02x01
- added U?: PBQ79616PAPTQ1, Snapeda:PAP0064F-IPC_A, symbol Snapeda:PBQ79616PAPTQ1
Connections:
- new net: C39.1, U?.38 (AVDD)
- new net: R41.1, R42.2
- new net: C36.1, U?.44 (NEG5V)
- new net: C40.1, U?.49 (DVDD)
- new net: C41.1, Q?.1 (C), R41.2
- new net: C38.1, U?.37 (REFHP)
- new net: J?.3 (Pin_3), U?.40 (COMLP)
- new net: J?.4 (Pin_4), U?.41 (COMLN)
- new net: J?.2 (Pin_2), U?.42 (COMHN)
- new net: J?.1 (Pin_1), U?.43 (COMHP)
- new net CB0: C1.1, C3.2, R1.2, U?.34 (CB0)
- new net CB1: C3.1, C5.2, R3.2, U?.32 (CB1)
- new net CB10: C21.1, C23.2, R21.2, U?.14 (CB10)
- new net CB11: C23.1, C25.2, R23.2, U?.12 (CB11)
- new net CB12: C25.1, C27.2, R25.2, U?.10 (CB12), U?.2 (CB16), U?.4 (CB15), U?.6 (CB14), U?.8 (CB13)
- new net CB13: C27.1, C29.2, R27.2
- new net CB14: C29.1, C31.2, R29.2
- new net CB15: C31.1, C33.2, R31.2
- new net CB16: C33.1, R33.2
- new net CB2: C5.1, C7.2, R5.2, U?.30 (CB2)
- new net CB3: C7.1, C9.2, R7.2, U?.28 (CB3)
- new net CB4: C11.2, C9.1, R9.2, U?.26 (CB4)
- new net CB5: C11.1, C13.2, R11.2, U?.24 (CB5)
- new net CB6: C13.1, C15.2, R13.2, U?.22 (CB6)
- new net CB7: C15.1, C17.2, R15.2, U?.20 (CB7)
- new net CB8: C17.1, C19.2, R17.2, U?.18 (CB8)
- new net CB9: C19.1, C21.2, R19.2, U?.16 (CB9)
- new net CEL13: R27.1, R28.1
- new net CELL0: J?.1 (Pin_1)
- new net CELL0S: J?.2 (Pin_2), R1.1, R2.1
- new net CELL1: R3.1, R4.1
- new net CELL10: R21.1, R22.1
- new net CELL11: R23.1, R24.1
- new net CELL12: R25.1, R26.1, R42.1, U?.1 (BAT)
- new net CELL14: R29.1, R30.1
- new net CELL15: R31.1, R32.1
- new net CELL16: R33.1, R34.1
- new net CELL2: R5.1, R6.1
- new net CELL3: R7.1, R8.1
- new net CELL4: R10.1, R9.1
- new net CELL5: R11.1, R12.1
- new net CELL6: R13.1, R14.1
- new net CELL7: R15.1, R16.1
- new net CELL8: R17.1, R18.1
- new net CELL9: R19.1, R20.1
- new net GND: C1.2, C2.2, C35.2, C36.2, C37.2, C38.2, C39.2, C40.2, C41.2, RT1.2 (Pin_2), RT2.2 (Pin_2), RT3.2 (Pin_2), RT4.2 (Pin_2), RT5.2 (Pin_2), RT6.2 (Pin_2), U?.36 (REFHM), U?.39 (AVSS), U?.46 (CVSS), U?.50 (DVSS), U?.65 (PAD)
- new net GPIO1: R35.2, RT1.1 (Pin_1), U?.61 (GPIO1)
- new net GPIO2: R36.2, RT2.1 (Pin_1), U?.60 (GPIO2)
- new net GPIO3: R37.2, RT3.1 (Pin_1), U?.59 (GPIO3)
- new net GPIO4: R38.2, RT4.1 (Pin_1), U?.58 (GPIO4)
- new net GPIO5: R39.2, RT5.1 (Pin_1), U?.57 (GPIO5)
- new net GPIO6: R40.2, RT6.1 (Pin_1), U?.56 (GPIO6)
- new net GPIO7: U?.55 (GPIO7)
- new net GPIO8: U?.54 (GPIO8)
- new net LDOIN: C37.1, Q?.3 (E), U?.47 (LDOIN)
- new net NPNB: Q?.2 (B), U?.48 (NPNB)
- new net TSREF: C35.1, R35.1, R36.1, R37.1, R38.1, R39.1, R40.1, U?.51 (TSREF)
- new net VC0: C2.1, C4.2, R2.2, U?.35 (VC0)
- new net VC1: C4.1, C6.2, R4.2, U?.33 (VC1)
- new net VC10: C22.1, C24.2, R22.2, U?.15 (VC10)
- new net VC11: C24.1, C26.2, R24.2, U?.13 (VC11)
- new net VC12: C26.1, C28.2, R26.2, U?.11 (VC12), U?.3 (VC16), U?.5 (VC15), U?.7 (VC14), U?.9 (VC13)
- new net VC13: C28.1, C30.2, R28.2
- new net VC14: C30.1, C32.2, R30.2
- new net VC15: C32.1, C34.2, R32.2
- new net VC16: C34.1, R34.2
- new net VC2: C6.1, C8.2, R6.2, U?.31 (VC2)
- new net VC3: C10.2, C8.1, R8.2, U?.29 (VC3)
- new net VC4: C10.1, C12.2, R10.2, U?.27 (VC4)
- new net VC5: C12.1, C14.2, R12.2, U?.25 (VC5)
- new net VC6: C14.1, C16.2, R14.2, U?.23 (VC6)
- new net VC7: C16.1, C18.2, R16.2, U?.21 (VC7)
- new net VC8: C18.1, C20.2, R18.2, U?.19 (VC8)
- new net VC9: C20.1, C22.2, R20.2, U?.17 (VC9)
- no-connect marks 0 -> 4
Other:
- note added: "CELLS"
- note added: "For future 16-cell build: remove short links and connect channels normally"
- note added: "GPIO7, GPIO8 are not used for the 12 CELLs design. But can be used for the 16 CELLs design"
- note added: "Middle module: COMH + COML used End module: one side used, other side terminated Ring: both sides active, terminate chain ends"
- note added: "Temp for CELL 2 CELL 4 CELL 6 CELL 8 CELL 10 CELL 12"
