File: Hardware/BMU/BMU-MCU.kicad_sch (KiCad schematic)
At the start: 6 parts, among them IC1 STM32C092RCT6, J6 Conn_ARM_JTAG_SWD_10

Commit message: add comment
Connections:
- no-connect marks 0 -> 51
Other:
- note added: "ALERT_SHUNT: Isolated overcurrent alert from shunt board to MCU GPIO/EXTI"
- note added: "| Function | MCU Pin | Notes | | ------------- | --------------- | ---------------------------------------- | | SWDIO | PA13 | Debug/programming | | SWCLK | PA14 | Debug/programming, shared with BOOT0 pin | | NRST | PF2 | Hardware reset | | BQ UART TX | PB6 | MCU → BQ79600 | | BQ UART RX | PB7 | BQ79600 → MCU | | Shunt I2C SCL | PB8 | I2C1_SCL | | Shunt I2C SDA | PB9 | I2C1_SDA | | CAN RX | PD0 |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"
- note removed: "Debug SWD"
- note removed: "Decoupling Capacitor"
- note removed: "Isolated overcurrent alert from shunt board to MCU GPIO/EXTI"
- note removed: "POWER"
- note removed: "RESET"
- moved on the sheet: C13, C15, C16, IC1, J6, R13

Commit message: add footprint
Parts:
- C13, C15, C16: footprint (none) -> Capacitor_SMD:C_0805_2012Metric
- IC1: footprint QFP50P1200X1200X160-64N -> STM32C092RCT6:QFP50P1200X1200X160-64N
- J6: footprint (none) -> Connector_PinHeader_1.27mm:PinHeader_2x05_P1.27mm_Vertical
- R13: footprint (none) -> Resistor_SMD:R_0805_2012Metric
Changed lines of the file:
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@@
 			)
 		)
-		(property "Footprint" ""
+		(property "Footprint" "Resistor_SMD:R_0805_2012Metric"
 			(at 184.15 100.33 0)
 			(hide yes)
@@
 			)
 		)
-		(property "Footprint" ""
+		(property "Footprint" "Connector_PinHeader_1.27mm:PinHeader_2x05_P1.27mm_Vertical"
 			(at 168.91 151.13 0)
 			(hide yes)
@@
 			)
 		)
-		(property "Footprint" "QFP50P1200X1200X160-64N"
+		(property "Footprint" "STM32C092RCT6:QFP50P1200X1200X160-64N"
 			(at 265.43 197.79 0)
 			(hide yes)
@@
 			)
 		)
-		(property "Footprint" ""
+		(property "Footprint" "Capacitor_SMD:C_0805_2012Metric"
 			(at 219.71 87.63 0)
 			(hide yes)
@@
 			)
 		)
-		(property "Footprint" ""
+		(property "Footprint" "Capacitor_SMD:C_0805_2012Metric"
 			(at 184.15 132.08 0)
 			(hide yes)
@@
 			)
 		)
-		(property "Footprint" ""
+		(property "Footprint" "Capacitor_SMD:C_0805_2012Metric"
 			(at 229.87 87.63 0)
 			(hide yes)

Commit message: update
Parts:
- renumbered C16 to C14
Changed lines of the file:
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@@
 		(in_pos_files yes)
 		(dnp no)
-		(property "Reference" "C16"
+		(property "Reference" "C14"
 			(at 215.138 85.852 0)
 			(show_name no)
@@
 			(project "BMU"
 				(path "/efb70416-ce55-4766-98ba-c3d23efcccb1/f115f1df-fd74-4b87-bcb3-90c9dd231c01"
-					(reference "C16")
+					(reference "C14")
 					(unit 1)
 				)

Commit message: update bmu
Connections:
- net STATUS_LED: now reaches IC1.30 (PB10)
- net SHUTDOWN_REQ: now reaches IC1.31 (PB11)
- no-connect marks 51 -> 49
Changed lines of the file:
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@@
-	)
-	(no_connect
-		(at 262.89 115.57)
 	)
 	(no_connect
@@
 	)
 	(no_connect
-		(at 262.89 113.03)
-	)
-	(no_connect
 		(at 262.89 180.34)
 	)
@@
 	(wire
 		(pts
+			(xy 264.16 115.57) (xy 262.89 115.57)
+		)
+		(stroke
+			(width 0)
+			(type default)
+		)
+	)
+	(wire
+		(pts
 			(xy 229.87 83.82) (xy 238.76 83.82)
 		)
@@
 	(wire
 		(pts
+			(xy 215.9 163.83) (xy 217.17 163.83)
+		)
+		(stroke
+			(width 0)
+			(type default)
+		)
+	)
+	(wire
+		(pts
 			(xy 238.76 83.82) (xy 238.76 96.52)
 		)
@@
 	(wire
 		(pts
+			(xy 215.9 161.29) (xy 217.17 161.29)
+		)
+		(stroke
+			(width 0)
+			(type default)
+		)
+	)
+	(wire
+		(pts
 			(xy 184.15 102.87) (xy 184.15 107.95)
 		)
@@
 	(wire
 		(pts
+			(xy 215.9 166.37) (xy 217.17 166.37)
+		)
+		(stroke
+			(width 0)
+			(type default)
+		)
+	)
+	(wire
+		(pts
 			(xy 163.83 170.18) (xy 165.1 170.18)
 		)
@@
 	(wire
 		(pts
+			(xy 264.16 113.03) (xy 262.89 113.03)
+		)
+		(stroke
+			(width 0)
+			(type default)
+		)
+	)
+	(wire
+		(pts
 			(xy 165.1 170.18) (xy 166.37 170.18)
 		)
@@
 		)
 	)
+	(hierarchical_label "STATUS_LED"
+		(shape output)
+		(at 264.16 115.57 0)
+		(effects
+			(font
+				(size 1.27 1.27)
+			)
+			(justify left)
+		)
+	)
 	(hierarchical_label "CAN_STBY"
 		(shape bidirectional)
-		(at 217.17 166.37 180)
+		(at 215.9 166.37 180)
 		(effects
 			(font
@@
 	(hierarchical_label "CAN_RX"
 		(shape bidirectional)
-		(at 217.17 161.29 180)
+		(at 215.9 161.29 180)
 		(effects
 			(font
@@
 	(hierarchical_label "CAN_TX"
 		(shape bidirectional)
-		(at 217.17 163.83 180)
+		(at 215.9 163.83 180)
 		(effects
 			(font
@@
 		)
 	)
+	(hierarchical_label "SHUTDOWN_REQ"
+		(shape output)
+		(at 264.16 113.03 0)
+		(effects
+			(font
+				(size 1.27 1.27)
+			)
+			(justify left)
+		)
+	)
