File: Hardware/BMU/BMU-COM Bridge.kicad_sch (KiCad schematic)
At the start: 9 parts, among them U4 BQ79600PWRQ1

Commit message: update bmu
Parts:
- added C18, C19, C20, C21, C22, C23: 100pF, Capacitor_SMD:C_0805_2012Metric, symbol Device:C
- added R10, R11, R12, R17, R26, R27, R28, R29: 0, Resistor_SMD:R_0805_2012Metric, symbol Device:R_US
- added R18, R19, R24, R25: 51, Resistor_SMD:R_0805_2012Metric, symbol Device:R_US
- added R20, R21, R22, R23: 499, Resistor_SMD:R_0805_2012Metric, symbol Device:R_US
- added T1, T3: CEP99-102, CEP99102, symbol CEP99-102:CEP99-102
- added U3, U6: PESD5V0L2BT, SOT23_NEX, symbol 2026-03-31_20-22-46:PESD5V0L2BT
Connections:
- net COMHN: now also U4.12 (COMHN), C22.1, R23.2, R25.2
- net COMHP: now also U4.13 (COMHP), C21.1, R22.1, R24.2
- net COMLN: now also U4.11 (COMLN), C19.1, R19.2, R21.2
- net COMLP: now also U4.10 (COMLP), C20.1, R18.2, R20.1
- net GND: now also C18.2, C19.2, C20.2, C21.2, C22.2, C23.2, R20.2, R21.1, R22.2, R23.1, U3.3, U6.3
- new net: R27.1, T3.1
- new net: R28.2, T3.5
- new net: R29.2, T3.8
- new net: R12.1, T1.8
- new net: R26.1, T3.4
- new net: C23.1, T3.2, T3.3
- new net: T3.6, T3.7
- new net: R11.2, T1.1
- new net: T1.2, T1.3
- new net: R10.2, T1.4
- new net: R17.1, T1.5
- new net: C18.1, T1.6, T1.7
- new net COMHN_1: R29.1
- new net COMHN_OPT: R25.1, R27.2, U6.2
- new net COMHP_1: R28.1
- new net COMHP_OPT: R24.1, R26.2, U6.1
- new net COMLN_2: R11.1
- new net COMLN_OPT: R12.2, R19.1, U3.1
- new net COMLP_2: R10.1
- new net COMLP_OPT: R17.2, R18.1, U3.2
Other:
- note added: "Tranformer Isolation For BQ79600"
- note removed: "ISO"
- moved on the sheet: C10, C11, C12, C9, R15, R7, R8, R9, U4

Commit message: layout
Parts:
- removed U3, U6: PESD5V0L2BT, SOT23_NEX, symbol 2026-03-31_20-22-46:PESD5V0L2BT
- added U8, U9: PESD5V0L2BT, PESD5V0L2BT:SOT23_NEX, symbol PESD5V0L2BT:PESD5V0L2BT
- T1: footprint CEP99102 -> CEP99-102:CEP99102
- T2: renamed from T3; footprint CEP99102 -> CEP99-102:CEP99102
Connections:
- net COMHN_OPT: now also U9.2
- net COMHP_OPT: now also U9.1
- net COMLN_OPT: now also U8.1
- net COMLP_OPT: now also U8.2
- net GND: now also U8.3, U9.3
