File: Hardware/BMU/BMU-POWER.kicad_sch (KiCad schematic)
At the start: 21 parts, among them Q2 AO3401A, U1 TPS54202DDC, U2 TLV75533PDBV

Commit message: add comment
Other:
- note added: "12 V input protection stage: F1 provides input fault protection. Q2 implements high-side reverse-polarity protection. D1 clamps input transients on the vehicle 12 V rail. D2 limits PMOS gate-source voltage. R6 pulls the gate low for normal turn-on."
- note removed: "12V Input"
- note removed: "Decoupling Capacitor"
- note removed: "Transient Voltage Suppressor"
- note removed: "reverse battery protection"
Changed lines of the file:
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@@
-		)
-	)
-	(rectangle
-		(start 88.9 110.49)
-		(end 113.03 123.19)
-		(stroke
-			(width 0)
-			(type default)
-		)
-		(fill
-			(type none)
-		)
-	)
-	(text "reverse battery protection"
-		(exclude_from_sim no)
-		(at 140.716 124.46 0)
-		(effects
-			(font
-				(size 1.27 1.27)
-			)
-		)
-	)
-	(text "Transient Voltage Suppressor"
-		(exclude_from_sim no)
-		(at 140.462 127.508 0)
-		(effects
-			(font
-				(size 1.27 1.27)
-			)
-		)
-	)
-	(text "Decoupling Capacitor"
-		(exclude_from_sim no)
-		(at 170.434 122.682 0)
-		(effects
-			(font
-				(size 1.27 1.27)
-			)
 		)
 	)
@@
 		)
 	)
-	(text "12V Input"
-		(exclude_from_sim no)
-		(at 100.33 116.84 0)
-		(effects
-			(font
-				(size 2.54 2.54)
-			)
-		)
-	)
 	(text "5V"
 		(exclude_from_sim no)
@@
 		)
 	)
-	(junction
-		(at 162.56 163.83)
-		(diameter 0)
-		(color 0 0 0 0)
+	(text "12 V input protection stage:\nF1 provides input fault protection.\nQ2 implements high-side reverse-polarity protection.\nD1 clamps input transients on the vehicle 12 V rail.\nD2 limits PMOS gate-source voltage.\nR6 pulls the gate low for normal turn-on."
+		(exclude_from_sim no)
+		(at 117.094 179.07 0)
+		(effects
+			(font
+				(size 1.27 1.27)
+			)
+			(justify left)
+		)
 	)
 	(junction
@@
 	)
 	(junction
+		(at 137.16 163.83)
+		(diameter 0)
+		(color 0 0 0 0)
+	)
+	(junction
 		(at 226.06 138.43)
 		(diameter 0)
@@
 	)
 	(junction
-		(at 264.16 163.83)
-		(diameter 0)
-		(color 0 0 0 0)
-	)
-	(junction
 		(at 162.56 135.89)
 		(diameter 0)
@@
 	)
 	(junction
-		(at 148.59 163.83)
-		(diameter 0)
-		(color 0 0 0 0)
-	)
-	(junction
 		(at 278.13 132.08)
 		(diameter 0)
@@
 		(color 0 0 0 0)
 	)
-	(junction
-		(at 278.13 163.83)
-		(diameter 0)
-		(color 0 0 0 0)
-	)
 	(wire
 		(pts
@@
 	(wire
 		(pts
-			(xy 264.16 163.83) (xy 278.13 163.83)
-		)
-		(stroke
-			(width 0)
-			(type default)
-		)
-	)
-	(wire
-		(pts
 			(xy 297.18 143.51) (xy 294.64 143.51)
 		)
@@
 	(wire
 		(pts
+			(xy 137.16 163.83) (xy 148.59 163.83)
+		)
+		(stroke
+			(width 0)
+			(type default)
+		)
+	)
+	(wire
+		(pts
 			(xy 214.63 135.89) (xy 218.44 135.89)
 		)
@@
 	(wire
 		(pts
-			(xy 148.59 163.83) (xy 162.56 163.83)
-		)
-		(stroke
-			(width 0)
-			(type default)
-		)
-	)
-	(wire
-		(pts
 			(xy 264.16 132.08) (xy 278.13 132.08)
 		)
@@
 	(wire
 		(pts
-			(xy 125.73 163.83) (xy 148.59 163.83)
+			(xy 125.73 163.83) (xy 137.16 163.83)
 		)
 		(stroke
@@
 	)
 	(symbol
+		(lib_id "power:GND")
+		(at 287.02 163.83 0)
+		(unit 1)
+		(body_style 1)
+		(exclude_from_sim no)
+		(in_bom yes)
+		(on_board yes)
+		(in_pos_files yes)
+		(dnp no)
+		(fields_autoplaced yes)
+		(property "Reference" "#PWR026"
+			(at 287.02 170.18 0)
+			(hide yes)
+			(show_name no)
+			(do_not_autoplace no)
+			(effects
+				(font
+					(size 1.27 1.27)
+				)
+			)
+		)
+		(property "Value" "GND"
+			(at 287.02 168.91 0)
+			(show_name no)
+			(do_not_autoplace no)
+			(effects
+				(font
+					(size 1.27 1.27)
+				)
+			)
+		)
+		(property "Footprint" ""
+			(at 287.02 163.83 0)
+			(hide yes)
+			(show_name no)
+			(do_not_autoplace no)
+			(effects
+				(font
+					(size 1.27 1.27)
+				)
+			)
+		)
+		(property "Datasheet" ""
+			(at 287.02 163.83 0)
+			(hide yes)
+			(show_name no)
+			(do_not_autoplace no)
+			(effects
+				(font
+					(size 1.27 1.27)
+				)
+			)
+		)
+		(property "Description" "Power symbol creates a global label with name \"GND\" , ground"
+			(at 287.02 163.83 0)
+			(hide yes)
+			(show_name no)
+			(do_not_autoplace no)
+			(effects
+				(font
+					(size 1.27 1.27)
+				)
+			)
+		)
+		(pin "1"
+		)
+		(instances
+			(project "BMU"
+				(path "/efb70416-ce55-4766-98ba-c3d23efcccb1/72276164-1341-4c36-b4e6-9b9f0edc7f8e"
+					(reference "#PWR026")
+					(unit 1)
+				)
+			)
+		)
+	)
+	(symbol
 		(lib_id "Device:C_Small")
 		(at 242.57 149.86 0)
@@
 					(unit 1)
 				)
+			)
+		)
+	)
+	(symbol
+		(lib_id "power:GND")
+		(at 137.16 163.83 0)
+		(unit 1)
+		(body_style 1)
+		(exclude_from_sim no)
+		(in_bom yes)
+		(on_board yes)
+		(in_pos_files yes)
+		(dnp no)
+		(fields_autoplaced yes)
+		(property "Reference" "#PWR027"
+			(at 137.16 170.18 0)
+			(hide yes)
+			(show_name no)
+			(do_not_autoplace no)
+			(effects
+				(font
+					(size 1.27 1.27)
+				)
+			)
+		)
+		(property "Value" "GND"
+			(at 137.16 168.91 0)
+			(show_name no)
+			(do_not_autoplace no)
+			(effects
+				(font
+					(size 1.27 1.27)
+				)
+			)
+		)
+		(property "Footprint" ""
+			(at 137.16 163.83 0)
+			(hide yes)
+			(show_name no)
+			(do_not_autoplace no)
+			(effects
+				(font
+					(size 1.27 1.27)
+				)
+			)
+		)
+		(property "Datasheet" ""
+			(at 137.16 163.83 0)
+			(hide yes)
+			(show_name no)
+			(do_not_autoplace no)
+			(effects
+				(font
+					(size 1.27 1.27)
+				)
+			)
+		)
+		(property "Description" "Power symbol creates a global label with name \"GND\" , ground"
+			(at 137.16 163.83 0)
+			(hide yes)
+			(show_name no)
+			(do_not_autoplace no)
+			(effects
+				(font
+					(size 1.27 1.27)
+				)
+			)
+		)
+		(pin "1"
+		)
+		(instances
+			(project "BMU"
+				(path "/efb70416-ce55-4766-98ba-c3d23efcccb1/72276164-1341-4c36-b4e6-9b9f0edc7f8e"
+					(reference "#PWR027")
+					(unit 1)
+				)

Commit message: add footprint
Parts:
- C1, C2, C6, C7, C8: footprint (none) -> Capacitor_SMD:C_0805_2012Metric
- C3, C4, C5: footprint (none) -> Capacitor_SMD:C_1206_3216Metric
- F1: footprint (none) -> Fuse:Fuse_1206_3216Metric
- L1: footprint (none) -> Inductor_SMD:L_7.3x7.3_H4.5
- R1, R2, R3, R4, R5, R6: footprint (none) -> Resistor_SMD:R_0805_2012Metric
Changed lines of the file:
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@@
 			)
 		)
-		(property "Footprint" ""
+		(property "Footprint" "Resistor_SMD:R_0805_2012Metric"
 			(at 264.16 135.89 0)
 			(hide yes)
@@
 			)
 		)
-		(property "Footprint" ""
+		(property "Footprint" "Capacitor_SMD:C_0805_2012Metric"
 			(at 171.45 151.13 0)
 			(hide yes)
@@
 			)
 		)
-		(property "Footprint" ""
+		(property "Footprint" "Fuse:Fuse_1206_3216Metric"
 			(at 120.65 137.668 90)
 			(hide yes)
@@
 			)
 		)
-		(property "Footprint" ""
+		(property "Footprint" "Resistor_SMD:R_0805_2012Metric"
 			(at 181.61 143.51 0)
 			(hide yes)
@@
 			)
 		)
-		(property "Footprint" ""
+		(property "Footprint" "Capacitor_SMD:C_1206_3216Metric"
 			(at 233.68 144.78 0)
 			(hide yes)
@@
 			)
 		)
-		(property "Footprint" ""
+		(property "Footprint" "Capacitor_SMD:C_0805_2012Metric"
 			(at 278.13 156.21 0)
 			(hide yes)
@@
 			)
 		)
-		(property "Footprint" ""
+		(property "Footprint" "Capacitor_SMD:C_0805_2012Metric"
 			(at 252.73 146.05 0)
 			(hide yes)
@@
 			)
 		)
-		(property "Footprint" ""
+		(property "Footprint" "Resistor_SMD:R_0805_2012Metric"
 			(at 181.61 157.48 0)
 			(hide yes)
@@
 			)
 		)
-		(property "Footprint" ""
+		(property "Footprint" "Resistor_SMD:R_0805_2012Metric"
 			(at 264.16 157.48 0)
 			(hide yes)
@@
 			)
 		)
-		(property "Footprint" ""
+		(property "Footprint" "Resistor_SMD:R_0805_2012Metric"
 			(at 264.16 144.78 0)
 			(hide yes)
@@
 			)
 		)
-		(property "Footprint" ""
+		(property "Footprint" "Capacitor_SMD:C_0805_2012Metric"
 			(at 220.98 135.89 0)
 			(hide yes)
@@
 			)
 		)
-		(property "Footprint" ""
+		(property "Footprint" "Capacitor_SMD:C_1206_3216Metric"
 			(at 242.57 149.86 0)
 			(hide yes)
@@
 			)
 		)
-		(property "Footprint" ""
+		(property "Footprint" "Inductor_SMD:L_7.3x7.3_H4.5"
 			(at 229.87 138.43 0)
 			(hide yes)
@@
 			)
 		)
-		(property "Footprint" ""
+		(property "Footprint" "Capacitor_SMD:C_0805_2012Metric"
 			(at 297.18 157.48 0)
 			(hide yes)
@@
 			)
 		)
-		(property "Footprint" ""
+		(property "Footprint" "Resistor_SMD:R_0805_2012Metric"
 			(at 148.59 158.75 0)
 			(hide yes)
@@
 			)
 		)
-		(property "Footprint" ""
+		(property "Footprint" "Capacitor_SMD:C_1206_3216Metric"
 			(at 162.56 146.05 0)
 			(hide yes)

Commit message: update bmu
Parts:
- removed D1: SMBJ16A, Diode_SMD:D_SMB, symbol Device:D
Changed lines of the file:
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@@
-	)
-	(junction
-		(at 137.16 163.83)
-		(diameter 0)
-		(color 0 0 0 0)
 	)
 	(junction
@@
 	)
 	(junction
-		(at 125.73 135.89)
-		(diameter 0)
-		(color 0 0 0 0)
-	)
-	(junction
 		(at 278.13 143.51)
 		(diameter 0)
@@
 	(wire
 		(pts
-			(xy 125.73 135.89) (xy 135.89 135.89)
-		)
-		(stroke
-			(width 0)
-			(type default)
-		)
-	)
-	(wire
-		(pts
 			(xy 114.3 134.62) (xy 114.3 135.89)
 		)
@@
 	(wire
 		(pts
-			(xy 124.46 135.89) (xy 125.73 135.89)
+			(xy 124.46 135.89) (xy 135.89 135.89)
 		)
 		(stroke
@@
 	(wire
 		(pts
-			(xy 137.16 163.83) (xy 148.59 163.83)
-		)
-		(stroke
-			(width 0)
-			(type default)
-		)
-	)
-	(wire
-		(pts
 			(xy 214.63 135.89) (xy 218.44 135.89)
 		)
@@
 	(wire
 		(pts
-			(xy 125.73 161.29) (xy 125.73 163.83)
-		)
-		(stroke
-			(width 0)
-			(type default)
-		)
-	)
-	(wire
-		(pts
 			(xy 287.02 163.83) (xy 297.18 163.83)
 		)
@@
 	(wire
 		(pts
-			(xy 125.73 163.83) (xy 137.16 163.83)
-		)
-		(stroke
-			(width 0)
-			(type default)
-		)
-	)
-	(wire
-		(pts
 			(xy 264.16 139.7) (xy 264.16 142.24)
 		)
@@
 		(pts
 			(xy 135.89 135.89) (xy 148.59 135.89)
-		)
-		(stroke
-			(width 0)
-			(type default)
-		)
-	)
-	(wire
-		(pts
-			(xy 125.73 135.89) (xy 125.73 153.67)
 		)
 		(stroke
@@
 	(symbol
 		(lib_id "power:GND")
-		(at 137.16 163.83 0)
+		(at 148.59 163.83 0)
 		(unit 1)
 		(body_style 1)
@@
 		(fields_autoplaced yes)
 		(property "Reference" "#PWR027"
-			(at 137.16 170.18 0)
+			(at 148.59 170.18 0)
 			(hide yes)
 			(show_name no)
@@
 		)
 		(property "Value" "GND"
-			(at 137.16 168.91 0)
+			(at 148.59 168.91 0)
 			(show_name no)
 			(do_not_autoplace no)
@@
 		)
 		(property "Footprint" ""
-			(at 137.16 163.83 0)
+			(at 148.59 163.83 0)
 			(hide yes)
 			(show_name no)
@@
 		)
 		(property "Datasheet" ""
-			(at 137.16 163.83 0)
+			(at 148.59 163.83 0)
 			(hide yes)
 			(show_name no)
@@
 		)
 		(property "Description" "Power symbol creates a global label with name \"GND\" , ground"
-			(at 137.16 163.83 0)
+			(at 148.59 163.83 0)
 			(hide yes)
 			(show_name no)
@@
 					(unit 1)
 				)
-			)
-		)
-	)
-	(symbol
-		(lib_id "Device:D")
-		(at 125.73 157.48 90)
-		(unit 1)
-		(body_style 1)
-		(exclude_from_sim no)
-		(in_bom yes)
-		(on_board yes)
-		(in_pos_files yes)
-		(dnp no)
-		(fields_autoplaced yes)
-		(property "Reference" "D1"
-			(at 128.27 156.2099 90)
-			(show_name no)
-			(do_not_autoplace no)
-			(effects
-				(font
-					(size 1.27 1.27)
-				)
-				(justify right)
-			)
-		)
-		(property "Value" "SMBJ16A"
-			(at 128.27 158.7499 90)
-			(show_name no)
-			(do_not_autoplace no)
-			(effects
-				(font
-					(size 1.27 1.27)
-				)
-				(justify right)
-			)
-		)
-		(property "Footprint" "Diode_SMD:D_SMB"
-			(at 125.73 157.48 0)
-			(hide yes)
-			(show_name no)
-			(do_not_autoplace no)
-			(effects
-				(font
-					(size 1.27 1.27)
-				)
-			)
-		)
-		(property "Datasheet" ""
-			(at 125.73 157.48 0)
-			(hide yes)
-			(show_name no)
-			(do_not_autoplace no)
-			(effects
-				(font
-					(size 1.27 1.27)
-				)
-			)
-		)
-		(property "Description" "Diode"
-			(at 125.73 157.48 0)
-			(hide yes)
-			(show_name no)
-			(do_not_autoplace no)
-			(effects
-				(font
-					(size 1.27 1.27)
-				)
-			)
-		)
-		(property "Sim.Device" "D"
-			(at 125.73 157.48 0)
-			(hide yes)
-			(show_name no)
-			(do_not_autoplace no)
-			(effects
-				(font
-					(size 1.27 1.27)
-				)
-			)
-		)
-		(property "Sim.Pins" "1=K 2=A"
-			(at 125.73 157.48 0)
-			(hide yes)
-			(show_name no)
-			(do_not_autoplace no)
-			(effects
-				(font
-					(size 1.27 1.27)
-				)
-			)
-		)
-		(pin "1"
-		)
-		(pin "2"
-		)
-		(instances
-			(project "BMU"
-				(path "/efb70416-ce55-4766-98ba-c3d23efcccb1/72276164-1341-4c36-b4e6-9b9f0edc7f8e"
-					(reference "D1")
-					(unit 1)
-				)

Commit message: layout
Parts:
- renumbered C3 to C1, C1 to C3
Connections:
- net at F1.2, Q2.2 (S): now also D2.1 (K); no longer D2.2 (A)
- net at Q2.1 (G), R6.1: now also D2.2 (A); no longer D2.1 (K)
Other:
- note added: "12 V input protection stage: F1 provides input fault protection. Q2 implements high-side reverse-polarity protection. D2 limits PMOS gate-source voltage. R6 pulls the gate low for normal turn-on."
- note removed: "12 V input protection stage: F1 provides input fault protection. Q2 implements high-side reverse-polarity protection. D1 clamps input transients on the vehicle 12 V rail. D2 limits PMOS gate-source voltage. R6 pulls the gate low for normal turn-on."
- moved on the sheet: D2, Q2
Changed lines of the file:
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@@
 	)
 	(rectangle
-		(start 190.5 109.22)
-		(end 214.63 121.92)
+		(start 191.77 109.22)
+		(end 215.9 121.92)
 		(stroke
 			(width 0)
@@
 	(text "5V"
 		(exclude_from_sim no)
-		(at 203.2 115.57 0)
+		(at 204.47 115.57 0)
 		(effects
 			(font
@@
 		)
 	)
-	(text "12 V input protection stage:\nF1 provides input fault protection.\nQ2 implements high-side reverse-polarity protection.\nD1 clamps input transients on the vehicle 12 V rail.\nD2 limits PMOS gate-source voltage.\nR6 pulls the gate low for normal turn-on."
-		(exclude_from_sim no)
-		(at 117.094 179.07 0)
+	(text "12 V input protection stage:\nF1 provides input fault protection.\nQ2 implements high-side reverse-polarity protection.\nD2 limits PMOS gate-source voltage.\nR6 pulls the gate low for normal turn-on."
+		(exclude_from_sim no)
+		(at 115.062 174.244 0)
 		(effects
 			(font
@@
 			(justify left)
 		)
+	)
+	(junction
+		(at 287.02 163.83)
+		(diameter 0)
+		(color 0 0 0 0)
+	)
+	(junction
+		(at 204.47 163.83)
+		(diameter 0)
+		(color 0 0 0 0)
+	)
+	(junction
+		(at 242.57 138.43)
+		(diameter 0)
+		(color 0 0 0 0)
+	)
+	(junction
+		(at 264.16 132.08)
+		(diameter 0)
+		(color 0 0 0 0)
+	)
+	(junction
+		(at 226.06 138.43)
+		(diameter 0)
+		(color 0 0 0 0)
+	)
+	(junction
+		(at 252.73 151.13)
+		(diameter 0)
+		(color 0 0 0 0)
+	)
+	(junction
+		(at 171.45 135.89)
+		(diameter 0)
+		(color 0 0 0 0)
+	)
+	(junction
+		(at 181.61 135.89)
+		(diameter 0)
+		(color 0 0 0 0)
+	)
+	(junction
+		(at 278.13 146.05)
+		(diameter 0)
+		(color 0 0 0 0)
+	)
+	(junction
+		(at 162.56 135.89)
+		(diameter 0)
+		(color 0 0 0 0)
+	)
+	(junction
+		(at 242.57 156.21)
+		(diameter 0)
+		(color 0 0 0 0)
+	)
+	(junction
+		(at 233.68 138.43)
+		(diameter 0)
+		(color 0 0 0 0)
+	)
+	(junction
+		(at 297.18 143.51)
+		(diameter 0)
+		(color 0 0 0 0)
+	)
+	(junction
+		(at 264.16 151.13)
+		(diameter 0)
+		(color 0 0 0 0)
+	)
+	(junction
+		(at 148.59 148.59)
+		(diameter 0)
+		(color 0 0 0 0)
+	)
+	(junction
+		(at 181.61 149.86)
+		(diameter 0)
+		(color 0 0 0 0)
+	)
+	(junction
+		(at 278.13 132.08)
+		(diameter 0)
+		(color 0 0 0 0)
+	)
+	(junction
+		(at 242.57 163.83)
+		(diameter 0)
+		(color 0 0 0 0)
+	)
+	(junction
+		(at 171.45 163.83)
+		(diameter 0)
+		(color 0 0 0 0)
+	)
+	(junction
+		(at 278.13 143.51)
+		(diameter 0)
+		(color 0 0 0 0)
 	)
 	(junction
@@
 	)
 	(junction
-		(at 287.02 163.83)
-		(diameter 0)
-		(color 0 0 0 0)
-	)
-	(junction
-		(at 204.47 163.83)
-		(diameter 0)
-		(color 0 0 0 0)
-	)
-	(junction
-		(at 242.57 138.43)
-		(diameter 0)
-		(color 0 0 0 0)
-	)
-	(junction
-		(at 264.16 132.08)
-		(diameter 0)
-		(color 0 0 0 0)
-	)
-	(junction
-		(at 226.06 138.43)
-		(diameter 0)
-		(color 0 0 0 0)
-	)
-	(junction
-		(at 252.73 151.13)
-		(diameter 0)
-		(color 0 0 0 0)
-	)
-	(junction
-		(at 171.45 135.89)
-		(diameter 0)
-		(color 0 0 0 0)
-	)
-	(junction
-		(at 181.61 135.89)
-		(diameter 0)
-		(color 0 0 0 0)
-	)
-	(junction
-		(at 278.13 146.05)
-		(diameter 0)
-		(color 0 0 0 0)
-	)
-	(junction
-		(at 162.56 135.89)
-		(diameter 0)
-		(color 0 0 0 0)
-	)
-	(junction
-		(at 242.57 156.21)
-		(diameter 0)
-		(color 0 0 0 0)
-	)
-	(junction
-		(at 233.68 138.43)
-		(diameter 0)
-		(color 0 0 0 0)
-	)
-	(junction
-		(at 297.18 143.51)
-		(diameter 0)
-		(color 0 0 0 0)
-	)
-	(junction
-		(at 264.16 151.13)
-		(diameter 0)
-		(color 0 0 0 0)
-	)
-	(junction
-		(at 148.59 147.32)
-		(diameter 0)
-		(color 0 0 0 0)
-	)
-	(junction
-		(at 181.61 149.86)
-		(diameter 0)
-		(color 0 0 0 0)
-	)
-	(junction
-		(at 278.13 132.08)
-		(diameter 0)
-		(color 0 0 0 0)
-	)
-	(junction
-		(at 242.57 163.83)
-		(diameter 0)
-		(color 0 0 0 0)
-	)
-	(junction
-		(at 171.45 163.83)
-		(diameter 0)
-		(color 0 0 0 0)
-	)
-	(junction
-		(at 278.13 143.51)
-		(diameter 0)
-		(color 0 0 0 0)
-	)
-	(junction
 		(at 264.16 139.7)
 		(diameter 0)
@@
 	(wire
 		(pts
-			(xy 143.51 147.32) (xy 148.59 147.32)
+			(xy 143.51 148.59) (xy 148.59 148.59)
 		)
 		(stroke
@@
 	(wire
 		(pts
+			(xy 148.59 148.59) (xy 148.59 156.21)
+		)
+		(stroke
+			(width 0)
+			(type default)
+		)
+	)
+	(wire
+		(pts
 			(xy 242.57 156.21) (xy 242.57 163.83)
 		)
@@
 	(wire
 		(pts
-			(xy 148.59 144.78) (xy 148.59 147.32)
+			(xy 154.94 135.89) (xy 154.94 153.67)
+		)
+		(stroke
+			(width 0)
+			(type default)
+		)
+	)
+	(wire
+		(pts
+			(xy 148.59 143.51) (xy 148.59 148.59)
 		)
 		(stroke
@@
 	(wire
 		(pts
-			(xy 154.94 135.89) (xy 154.94 152.4)
-		)
-		(stroke
-			(width 0)
-			(type default)
-		)
-	)
-	(wire
-		(pts
 			(xy 264.16 147.32) (xy 264.16 151.13)
 		)
@@
 	(wire
 		(pts
-			(xy 148.59 135.89) (xy 148.59 137.16)
-		)
-		(stroke
-			(width 0)
-			(type default)
-		)
-	)
-	(wire
-		(pts
 			(xy 181.61 135.89) (xy 171.45 135.89)
 		)
@@
 	(wire
 		(pts
-			(xy 135.89 135.89) (xy 135.89 142.24)
-		)
-		(stroke
-			(width 0)
-			(type default)
-		)
-	)
-	(wire
-		(pts
-			(xy 135.89 152.4) (xy 154.94 152.4)
+			(xy 135.89 135.89) (xy 135.89 143.51)
+		)
+		(stroke
+			(width 0)
+			(type default)
+		)
+	)
+	(wire
+		(pts
+			(xy 135.89 153.67) (xy 154.94 153.67)
 		)
 		(stroke
@@
 		(pts
 			(xy 181.61 163.83) (xy 204.47 163.83)
-		)
-		(stroke
-			(width 0)
-			(type default)
-		)
-	)
-	(wire
-		(pts
-			(xy 148.59 147.32) (xy 148.59 156.21)
 		)
 		(stroke
@@
 	(symbol
 		(lib_id "Transistor_FET:AO3401A")
-		(at 138.43 147.32 180)
+		(at 138.43 148.59 180)
 		(unit 1)
 		(body_style 1)
@@
 		(fields_autoplaced yes)
 		(property "Reference" "Q2"
-			(at 132.08 146.0499 0)
+			(at 132.08 147.3199 0)
 			(show_name no)
 			(do_not_autoplace no)
@@
 		)
 		(property "Value" "AO3401A"
-			(at 132.08 148.5899 0)
+			(at 132.08 149.8599 0)
 			(show_name no)
 			(do_not_autoplace no)
@@
 		)
 		(property "Footprint" "Package_TO_SOT_SMD:SOT-23"
-			(at 133.35 145.415 0)
+			(at 133.35 146.685 0)
 			(hide yes)
 			(show_name no)
@@
 		)
 		(property "Datasheet" "http://www.aosmd.com/pdfs/datasheet/AO3401A.pdf"
-			(at 133.35 143.51 0)
+			(at 133.35 144.78 0)
 			(hide yes)
 			(show_name no)
@@
 		)
 		(property "Description" "-4.0A Id, -30V Vds, P-Channel MOSFET, SOT-23"
-			(at 138.43 147.32 0)
+			(at 138.43 148.59 0)
 			(hide yes)
 			(show_name no)
@@
 	(symbol
 		(lib_id "Device:D_Zener")
-		(at 148.59 140.97 90)
+		(at 148.59 139.7 270)
 		(unit 1)
 		(body_style 1)
@@
 		(dnp no)
 		(property "Reference" "D2"
-			(at 143.764 141.986 90)
+			(at 151.638 137.16 90)
 			(show_name no)
 			(do_not_autoplace no)
@@
 		)
 		(property "Value" "BZT52-C15"
-			(at 136.652 138.43 90)
+			(at 148.59 142.494 90)
 			(show_name no)
 			(do_not_autoplace no)
@@
 		)
 		(property "Footprint" "Diode_SMD:D_SOD-123"
-			(at 148.59 140.97 0)
+			(at 148.59 139.7 0)
 			(hide yes)
 			(show_name no)
@@
 		)
 		(property "Datasheet" ""
-			(at 148.59 140.97 0)
+			(at 148.59 139.7 0)
 			(hide yes)
 			(show_name no)
@@
 		)
 		(property "Description" "Zener diode"
-			(at 148.59 140.97 0)
+			(at 148.59 139.7 0)
 			(hide yes)
 			(show_name no)
@@
 		(dnp no)
 		(fields_autoplaced yes)
-		(property "Reference" "C1"
+		(property "Reference" "C3"
 			(at 220.9863 129.54 90)
 			(show_name no)
@@
 			(project "BMU"
 				(path "/efb70416-ce55-4766-98ba-c3d23efcccb1/72276164-1341-4c36-b4e6-9b9f0edc7f8e"
-					(reference "C1")
+					(reference "C3")
 					(unit 1)
 				)
@@
 		(dnp no)
 		(fields_autoplaced yes)
-		(property "Reference" "C3"
+		(property "Reference" "C1"
 			(at 165.1 144.7862 0)
 			(show_name no)
@@
 			(project "BMU"
 				(path "/efb70416-ce55-4766-98ba-c3d23efcccb1/72276164-1341-4c36-b4e6-9b9f0edc7f8e"
-					(reference "C3")
+					(reference "C1")
 					(unit 1)
 				)
