File: Hardware/BMU/BMU.kicad_pcb (KiCad board)
At the start: 4 copper layers, 47 parts, among them IC1 STM32C092RCT6, J1 IN/GND, J2 COM, J3 I2C, J4 CAN, J5 SHUNT, J6 Conn_ARM_JTAG_SWD_10, Q2 AO3401A, U1 TPS54202DDC, U2 TLV75533PDBV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

Commit message: update
Parts:
- moved C1 53.9 mm to (188.6, 77.5)
- moved C2 53.9 mm to (188.5, 80.5)
- moved C3 49.1 mm to (188.4, 83.5)
- moved C4 49.1 mm to (188.4, 86.8)
- moved C5 49.1 mm to (188.4, 90.2)
- moved R1 48.9 mm to (179.0, 80.1)
- moved R2 48.9 mm to (179.0, 83.0)
- moved R3 48.9 mm to (179.0, 86.0)
- moved R4 48.9 mm to (179.0, 89.0)
- moved R5 48.9 mm to (179.0, 91.9)
- moved R6 48.9 mm to (179.0, 94.8)
- moved C6 48.8 mm to (183.4, 84.0)
- moved C7 48.8 mm to (183.4, 87.0)
- moved C8 48.8 mm to (183.4, 90.0)
- moved F1 48.0 mm to (183.4, 80.3)
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- renumbered C16 to C14, C14 to C16
Connections:
- net /BMU-BQ79600/FAULT_N renamed /BMU-COM Bridge/FAULT_N
- net /BMU-BQ79600/MISO/TX renamed /BMU-COM Bridge/MISO/TX
- net /BMU-BQ79600/MOSI/RX renamed /BMU-COM Bridge/MOSI/RX
- J2 pad 1: /J2_COMLN -> /COMLN
- J2 pad 2: /J2_COMLP -> /COMLP
- J2 pad 3: /J2_COMHN -> /COMHN
- J2 pad 4: /J2_COMHP -> /COMHP
- U4 pad 10: /J2_COMLP -> Net-(U4-COMHN)
- U4 pad 11: /J2_COMLN -> Net-(U4-COMHN)
- U4 pad 12: /J2_COMHN -> Net-(U4-COMHN)
- U4 pad 13: /J2_COMHP -> Net-(U4-COMHN)

Commit message: layout
Parts:
- removed D1: SMBJ16A, Diode_SMD:D_SMB
- added C18: 100pF, Capacitor_SMD:C_0805_2012Metric, F.Cu at (118.2, 119.7)
- added C19: 100pF, Capacitor_SMD:C_0805_2012Metric, F.Cu at (141.2, 112.2)
- added C20: 100pF, Capacitor_SMD:C_0805_2012Metric, F.Cu at (141.2, 126.2)
- added C21: 100pF, Capacitor_SMD:C_0805_2012Metric, F.Cu at (141.2, 83.7)
- added C22: 100pF, Capacitor_SMD:C_0805_2012Metric, F.Cu at (141.2, 97.7)
- added C23: 100pF, Capacitor_SMD:C_0805_2012Metric, F.Cu at (118.2, 91.2)
- added J4: LOW SIDE, 70551-0038:CONN_70551-xxxx_04_MOL, F.Cu at (94.8, 122.4)
- added J8: AUX_IO, Connector_PinHeader_2.54mm:PinHeader_1x02_P2.54mm_Vertical, F.Cu at (219.3, 135.7)
- added R10: 0, Resistor_SMD:R_0805_2012Metric, F.Cu at (97.8, 118.2)
- added R11: 0, Resistor_SMD:R_0805_2012Metric, F.Cu at (97.8, 115.7)
- added R12: 0, Resistor_SMD:R_0805_2012Metric, F.Cu at (118.2, 116.2)
- added R17: 0, Resistor_SMD:R_0805_2012Metric, F.Cu at (118.2, 123.2)
- added R18: 51, Resistor_SMD:R_0805_2012Metric, F.Cu at (140.7, 123.2)
- added R19: 51, Resistor_SMD:R_0805_2012Metric, F.Cu at (140.7, 116.2)
- added R20: 499, Resistor_SMD:R_0805_2012Metric, F.Cu at (148.2, 123.7)
- added R21: 499, Resistor_SMD:R_0805_2012Metric, F.Cu at (147.8, 117.7)
- added R22: 499, Resistor_SMD:R_0805_2012Metric, F.Cu at (146.2, 89.2)
- added R23: 499, Resistor_SMD:R_0805_2012Metric, F.Cu at (147.2, 94.7)
- added R24: 51, Resistor_SMD:R_0805_2012Metric, F.Cu at (140.7, 87.7)
- added R25: 51, Resistor_SMD:R_0805_2012Metric, F.Cu at (140.7, 94.7)
- added R26: 0, Resistor_SMD:R_0805_2012Metric, F.Cu at (118.2, 87.7)
- added R27: 0, Resistor_SMD:R_0805_2012Metric, F.Cu at (118.2, 94.7)
- added R28: 0, Resistor_SMD:R_0805_2012Metric, F.Cu at (97.8, 92.7)
- added R29: 0, Resistor_SMD:R_0805_2012Metric, F.Cu at (97.7, 95.2)
- added T1: CEP99-102, CEP99-102:CEP99102, F.Cu at (108.6, 119.7)
- added T2: CEP99-102, CEP99-102:CEP99102, F.Cu at (108.6, 91.2)
- added U8: PESD5V0L2BT, PESD5V0L2BT:SOT23_NEX, F.Cu at (141.1, 119.2)
- added U9: PESD5V0L2BT, PESD5V0L2BT:SOT23_NEX, F.Cu at (141.1, 90.8)
- J2: value COM -> HIGH SIDE; footprint Connector_PinHeader_2.54mm:PinHeader_1x04_P2.54mm_Vertical -> 70551-0038:CONN_70551-xxxx_04_MOL
- moved U2 46.2 mm to (203.1, 74.7)
- moved F1 32.6 mm to (151.2, 75.2)
- moved R6 32.3 mm to (150.8, 79.2)
- moved C7 30.2 mm to (210.2, 73.2)
- moved C8 30.2 mm to (210.2, 76.2)
- moved J2 29.4 mm to (94.8, 96.4), turned to -90 degrees
- moved J1 28.1 mm to (150.0, 70.7), turned to 90 degrees
- moved L1 24.6 mm to (190.4, 73.7)
- moved U4 24.4 mm to (155.8, 107.2), turned to -90 degrees
- moved C9 24.0 mm to (155.2, 115.7)
- moved R15 22.5 mm to (158.7, 113.2)
- moved J6 22.3 mm to (169.5, 135.4)
- moved C2 22.3 mm to (166.7, 75.7)
- moved C1 22.3 mm to (166.6, 78.7)
- moved R3 20.0 mm to (197.2, 77.7)
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- renumbered C3 to C1, C1 to C3, J4 to J7
Connections:
- D2 pad 2: Net-(D1-A) -> Net-(D2-A)
- F1 pad 2: Net-(D1-A) -> Net-(D2-K)
- IC1 pad 30: unconnected-(IC1-PB10-Pad30) -> /BMU-MCU/STATUS_LED
- IC1 pad 31: unconnected-(IC1-PB11-Pad31) -> /BMU-MCU/SHUTDOWN_REQ
- IC1 pad 50: /BMU-MCU/CAN_RX -> /BMU-CAN/CAN_RX
- IC1 pad 51: /BMU-MCU/CAN_TX -> /BMU-CAN/CAN_TX
- J2 pad 1: /COMLN -> unconnected-(J2-Pad1)
- J2 pad 2: /COMLP -> unconnected-(J2-Pad2)
- J2 pad 3: /COMHN -> /High COMHP
- J2 pad 4: /COMHP -> /High COMHN
- Q2 pad 1: Net-(D2-K) -> Net-(D2-A)
- Q2 pad 2: Net-(D1-A) -> Net-(D2-K)
- R6 pad 1: Net-(D2-K) -> Net-(D2-A)
- U4 pad 10: Net-(U4-COMHN) -> COMLP
- U4 pad 11: Net-(U4-COMHN) -> COMLN
- U4 pad 12: Net-(U4-COMHN) -> COMHN
- U4 pad 13: Net-(U4-COMHN) -> COMHP
Routing:
- net /BMU-COM Bridge/COMLP_OPT: track 0.00 -> 23.8 mm
- net /BMU-COM Bridge/COMHN_OPT: track 0.00 -> 23.8 mm
- net /BMU-COM Bridge/COMHP_OPT: track 0.00 -> 22.9 mm
- net /BMU-COM Bridge/COMLN_OPT: track 0.00 -> 22.8 mm
- net Net-(R28-Pad2): track 0.00 -> 7.49 mm
- net Net-(R10-Pad2): track 0.00 -> 7.24 mm
- net Net-(C18-Pad1): track 0.00 -> 6.32 mm
- net Net-(R29-Pad2): track 0.00 -> 5.13 mm
- net Net-(R11-Pad2): track 0.00 -> 5.04 mm
- net COMLN: track 0.00 -> 3.87 mm
- net Net-(R27-Pad1): track 0.00 -> 3.44 mm
- net Net-(R26-Pad1): track 0.00 -> 3.44 mm
- net Net-(R17-Pad1): track 0.00 -> 3.44 mm
- net Net-(R12-Pad1): track 0.00 -> 3.44 mm
- net COMHP: track 0.00 -> 3.27 mm
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Other:
- board text added: "VIKING MOTOR SPORTS (VMS) BATTERY MANAGEMENT UNIT (BMU) 2026.4"
